File: Swarmy_INS_Flight_Controller/Swarmy_INS_Flight_Controller.brd (EAGLE design)
At the start: 96 x 96 mm, 144 parts, among them J1 MICRO-SD-SDIOPUSH-PUSH, Q1 20V/4.2A/52mΩ/1.4W, Q2 20V/4.2A/52mΩ/1.4W, Q3 BCF81SMD, Q4 BCF81SMD, Q5 BCF81SMD, Q7 BCF81SMD

Commit message: Final Form
Parts:
- added D3, D4: GREEN, SparkFun-LED:LED-0603
- added D7: 120mA/40V/370mV, SparkFun-DiscreteSemi:SOD-523
- added Q6: BCF81SMD, transistor-npn:SOT23-BEC
- added R16: 220R, SparkFun-Resistors:0603
- added R21, R22: 10k, SparkFun-Resistors:0603
- added U$80: (no value), PASIVE_BUZZER_5MM_X_5MM_20MM:PASIVE_BUZZER_5MM_X_5MM_20MM
- added U$81, U$82, U$83, U$84, U$85, U$86: 2X2MM_SQUARE_PAD, 2x2mm_square_pad_SM:2X2MM_SQUARE_PAD
- moved U$59 9.00 mm to (94.0, 81.0)
- moved U$63 9.00 mm to (94.0, 72.0)
- moved R3 8.99 mm to (18.0, 58.2)
- moved R20 6.00 mm to (24.0, 58.1)
- moved R9 6.00 mm to (27.0, 58.1)
- moved R14 5.45 mm to (63.0, 64.5)
- moved U$29 3.01 mm to (43.0, 81.0)
- moved R2 3.00 mm to (21.0, 58.1)
- moved U$39 3.00 mm to (21.0, 53.0)
- moved U$40 3.00 mm to (18.0, 53.0)
- moved U$41 3.00 mm to (33.0, 53.0)
- moved U$42 3.00 mm to (30.0, 53.0)
- moved U$50 3.00 mm to (94.0, 81.0)
- moved U$51 3.00 mm to (94.0, 84.0)
- moved U$58 3.00 mm to (94.0, 78.0)
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Connections:
- new net BUZ_PIN: R16.2, U$44.IO-2
- new net GPIO_2: U$13.IO-2, U$86.1
- new net GPIO_25: U$13.IO-25, U$81.1
- new net GPIO_26: U$13.IO-26, U$82.1
- new net GPIO_27: U$13.IO-27, U$83.1
- new net GPIO_34: U$13.IO-34, U$84.1
- new net GPIO_35: U$13.IO-35, U$85.1
- new net N$10: Q6.B, R16.1
- new net N$12: D7.C, Q6.E, U$80.+
- new net N$6: D3.A, R21.1
- new net N$7: D4.A, R22.1
- new net N$8: D3.C, U$43.1
- new net N$9: D4.C, U$49.1
- new net SD_CS: J1.CS/DAT3, U$44.IO-5
- net 3.3V_OUT_1: now also R21.2
- net 3.3V_OUT_2: now also J1.VCC, Q6.C, R22.2
- net GND: now also D7.A, J1.GND, J1.GND1, J1.GND3, U$80.-
- net MISO_3: now also J1.DO/DAT0
- net MOSI_3: now also J1.DI/CMD
- net SCL_2: now also R3.2; no longer R2.2
- net SDA_2: now also R2.2; no longer R3.2
- net SPI_CLK_3: now also J1.SCLK
- net SPI_CS_3: now also U$44.IO-4; no longer U$44.IO-5
Routing:
- net S2: track 0.00 -> 171.3 mm, vias 0 -> 8
- net GND: track 162.0 -> 308.2 mm, vias 54 -> 68
- net 3.3V_OUT_1: track 0.00 -> 93.6 mm, vias 0 -> 2
- net 3.3V_OUT_2: track 0.00 -> 76.7 mm, vias 0 -> 2
- net MOSI_3: track 0.00 -> 60.9 mm, vias 0 -> 2
- net SPI_CLK_3: track 0.00 -> 52.0 mm, vias 0 -> 2
- net MISO_3: track 0.00 -> 51.9 mm, vias 0 -> 2
- net SCL_1: track 0.00 -> 49.1 mm, vias 0 -> 4
- net M_SIG_RB: track 0.00 -> 46.4 mm, vias 0 -> 2
- net SDA_1: track 0.00 -> 43.7 mm, vias 0 -> 2
- net EN_2: track 0.00 -> 41.4 mm
- net EN_1: track 0.00 -> 40.6 mm
- net TX_1: track 0.00 -> 39.4 mm, vias 0 -> 2
- net SPI_CLK_4: track 0.00 -> 38.9 mm, vias 0 -> 2
- net SDA_2: track 0.00 -> 38.8 mm, vias 0 -> 2
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- added copper zone on layer 1, net 3.3V_OUT_1
- added copper zone on layer 1, net 3.3V_OUT_2
- added copper zone on layer 16, net GND
Other:
- outline, holes or cut-outs redrawn
- board text added: "0x0D"
- board text added: "0x6A"
- board text added: "0x76"
- board text added: "0x77"
- board text added: "2"
- board text added: "25"
- board text added: "26"
- board text added: "27"
- board text added: "34"
- board text added: "35"
- board text added: "3V3"
- board text added: "CLK14"
- board text added: "CLK18"
- board text added: "CS15"
- board text added: "CS4"
- board text added: "CS5"
- board text added: "JLCJLCJLCJLC"
- board text added: "MISO12"
- board text added: "MISO19"
- board text added: "MOSI13"
- board text added: "MOSI23"
- board text added: "Micro SD"
- board text added: "RX16"
- board text added: "S25"
- board text added: "S26"
- board text added: "S27"
- board text added: "S35"
- board text added: "SCL22"
- board text added: "SCL32"
- board text added: "SDA21"
- board text added: "SDA33"
- board text added: "SPI"
- board text added: "TX17"
- board text added: "X"
- board text added: "Y"
- board text added: "Z"
- board text removed: "1-3S"
- board text removed: "BAT +"
- board text removed: "BAT -"
- board text removed: "CLK1"
- board text removed: "CLK2"
- board text removed: "CS1"
- board text removed: "CS2"
- board text removed: "MISO1"
- board text removed: "MISO2"
- board text removed: "MOSI1"
- board text removed: "MOSI2"
- board text removed: "S1"
- board text removed: "S2"
- board text removed: "S3"
- board text removed: "S4"
