File: Swarmy_INS_Flight_Controller/Swarmy_INS_Flight_Controller.sch (EAGLE design)
At the start: 144 parts, among them J1 MICRO-SD-SDIOPUSH-PUSH, Q1 20V/4.2A/52mΩ/1.4W, Q2 20V/4.2A/52mΩ/1.4W, Q3 BCF81SMD, Q4 BCF81SMD, Q5 BCF81SMD, Q7 BCF81SMD

Commit message: Final Form
Parts:
- added D3, D4: GREEN, SparkFun-LED:LED-GREEN0603
- added D7: 120mA/40V/370mV, SparkFun-DiscreteSemi:DIODE-SCHOTTKY-RB751S40
- added Q6: BCF81SMD, transistor-npn:BCF81SMD
- added R16: 220R, SparkFun-Resistors:12KOHM-0603-1/10W-1%
- added R21, R22: 10k, SparkFun-Resistors:12KOHM-0603-1/10W-1%
- added U$80: (no value), PASIVE_BUZZER_5MM_X_5MM_20MM:PASIVE_BUZZER_5MM_X_5MM_20MM
- added U$81, U$82, U$83, U$84, U$85, U$86: 2X2MM_SQUARE_PAD, 2x2mm_square_pad_SM:2X2MM_SQUARE_PAD
Connections:
- new net BUZ_PIN: R16.2, U$44.IO-2
- new net GPIO_2: U$13.IO-2, U$86.1
- new net GPIO_25: U$13.IO-25, U$81.1
- new net GPIO_26: U$13.IO-26, U$82.1
- new net GPIO_27: U$13.IO-27, U$83.1
- new net GPIO_34: U$13.IO-34, U$84.1
- new net GPIO_35: U$13.IO-35, U$85.1
- new net N$10: Q6.B, R16.1
- new net N$12: D7.C, Q6.E, U$80.+
- new net N$6: D3.A, R21.1
- new net N$7: D4.A, R22.1
- new net N$8: D3.C, U$43.1
- new net N$9: D4.C, U$49.1
- new net SD_CS: J1.DAT3/!CS!, U$44.IO-5
- net 3.3V_OUT_1: now also R21.2
- net 3.3V_OUT_2: now also J1.VCC, Q6.C, R22.2
- net GND: now also D7.A, J1.GND, U$80.-
- net MISO_3: now also J1.DAT0/SDO
- net MOSI_3: now also J1.CMD/SDI
- net SCL_2: now also R3.2; no longer R2.2
- net SDA_2: now also R2.2; no longer R3.2
- net SPI_CLK_3: now also J1.CLK/SCK
- net SPI_CS_3: now also U$44.IO-4; no longer U$44.IO-5
Other:
- moved on the sheet: C21, C22, C23, C24, C25, C26, C27, C28, C29, C30, C31, C32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
